Commit message: Added Materials for More Accurate Simulation

File: virtual_gamefield/roboken_world/urdf/robot.urdf (robot description, URDF)
Before this commit: robot onshape, 1 links, 0 joints
Links:
- link gamefield: mass 0 -> 247.11182957758143175; geometry collision mesh filename=package:///blue_wheel.stl; collision mesh filename=package:///cabin.stl
